File: keyboardProject/keyboardProject.sch (KiCad schematic (older format))
At the start: 24 parts, among them K1 KEYSW, K2 KEYSW, K3 KEYSW, K4 KEYSW

Commit message: annotate schematic
Parts:
- gave numbers to parts that had none: 16
Changed lines of the file:
@@
 $EndDescr
 $Comp
-L keyboardParts:ATMEGA32U4 U?
+L keyboardParts:ATMEGA32U4 U1
 U 1 1 5F21E47E
 P 4500 3850
-F 0 "U?" H 4525 5187 60  0000 C CNN
+F 0 "U1" H 4525 5187 60  0000 C CNN
 F 1 "ATMEGA32U4" H 4525 5081 60  0000 C CNN
 F 2 "" H 4500 3850 60  0000 C CNN
@@
 $EndComp
 $Comp
-L keyboardParts:XTAL_GND X?
+L keyboardParts:XTAL_GND X1
 U 1 1 5F21EF91
 P 2400 4500
-F 0 "X?" H 2400 4792 60  0000 C CNN
+F 0 "X1" H 2400 4792 60  0000 C CNN
 F 1 "XTAL_GND" H 2400 4686 60  0000 C CNN
 F 2 "" H 2400 4500 60  0000 C CNN
@@
 $EndComp
 $Comp
-L Device:C_Small C?
+L Device:C_Small C6
 U 1 1 5F220920
 P 2700 4650
-F 0 "C?" H 2792 4696 50  0000 L CNN
+F 0 "C6" H 2792 4696 50  0000 L CNN
 F 1 "22p" H 2792 4605 50  0000 L CNN
 F 2 "" H 2700 4650 50  0001 C CNN
@@
 $EndComp
 $Comp
-L Device:C_Small C?
+L Device:C_Small C3
 U 1 1 5F2211C7
 P 2100 4650
-F 0 "C?" H 2192 4696 50  0000 L CNN
+F 0 "C3" H 2192 4696 50  0000 L CNN
 F 1 "22p" H 2192 4605 50  0000 L CNN
 F 2 "" H 2100 4650 50  0001 C CNN
@@
 Connection ~ 2700 4500
 $Comp
-L power:VCC #PWR?
+L power:VCC #PWR0101
 U 1 1 5F235AC0
 P 1400 1450
-F 0 "#PWR?" H 1400 1300 50  0001 C CNN
+F 0 "#PWR0101" H 1400 1300 50  0001 C CNN
 F 1 "VCC" H 1415 1623 50  0000 C CNN
 F 2 "" H 1400 1450 50  0001 C CNN
@@
 $EndComp
 $Comp
-L Device:C C?
+L Device:C C1
 U 1 1 5F235FDD
 P 1400 1700
-F 0 "C?" H 1515 1746 50  0000 L CNN
+F 0 "C1" H 1515 1746 50  0000 L CNN
 F 1 "0.1u" H 1515 1655 50  0000 L CNN
 F 2 "" H 1438 1550 50  0001 C CNN
@@
 $EndComp
 $Comp
-L Device:C C?
+L Device:C C2
 U 1 1 5F237A95
 P 1800 1700
-F 0 "C?" H 1915 1746 50  0000 L CNN
+F 0 "C2" H 1915 1746 50  0000 L CNN
 F 1 "0.1u" H 1915 1655 50  0000 L CNN
 F 2 "" H 1838 1550 50  0001 C CNN
@@
 $EndComp
 $Comp
-L Device:C C?
+L Device:C C4
 U 1 1 5F2382E6
 P 2200 1700
-F 0 "C?" H 2315 1746 50  0000 L CNN
+F 0 "C4" H 2315 1746 50  0000 L CNN
 F 1 "0.1u" H 2315 1655 50  0000 L CNN
 F 2 "" H 2238 1550 50  0001 C CNN
@@
 $EndComp
 $Comp
-L Device:C C?
+L Device:C C5
 U 1 1 5F23882A
 P 2600 1700
-F 0 "C?" H 2715 1746 50  0000 L CNN
+F 0 "C5" H 2715 1746 50  0000 L CNN
 F 1 "0.1u" H 2715 1655 50  0000 L CNN
 F 2 "" H 2638 1550 50  0001 C CNN
@@
 $EndComp
 $Comp
-L Device:C C?
+L Device:C C7
 U 1 1 5F239C38
 P 3000 1700
-F 0 "C?" H 3115 1746 50  0000 L CNN
+F 0 "C7" H 3115 1746 50  0000 L CNN
 F 1 "4.7u" H 3115 1655 50  0000 L CNN
 F 2 "" H 3038 1550 50  0001 C CNN
@@
 	1800 1900 2200 1900
 $Comp
-L keyboardParts:SW_PUSH SW?
+L keyboardParts:SW_PUSH SW1
 U 1 1 5F23E104
 P 2400 4000
-F 0 "SW?" H 2400 4255 50  0000 C CNN
+F 0 "SW1" H 2400 4255 50  0000 C CNN
 F 1 "SW_PUSH" H 2400 4164 50  0000 C CNN
 F 2 "" H 2400 4000 60  0000 C CNN
@@
 $EndComp
 $Comp
-L Device:R R?
+L Device:R R1
 U 1 1 5F242DF7
 P 2400 3650
-F 0 "R?" V 2193 3650 50  0000 C CNN
+F 0 "R1" V 2193 3650 50  0000 C CNN
 F 1 "10k" V 2284 3650 50  0000 C CNN
 F 2 "" V 2330 3650 50  0001 C CNN
@@
 	2100 4000 2000 4000
 $Comp
-L power:VCC #PWR?
+L power:VCC #PWR0102
 U 1 1 5F248CB6
 P 2150 3650
-F 0 "#PWR?" H 2150 3500 50  0001 C CNN
+F 0 "#PWR0102" H 2150 3500 50  0001 C CNN
 F 1 "VCC" V 2165 3777 50  0000 L CNN
 F 2 "" H 2150 3650 50  0001 C CNN
@@
 	2250 3650 2150 3650
 $Comp
-L Device:R R?
+L Device:R R4
 U 1 1 5F24C974
 P 6150 3900
-F 0 "R?" V 5943 3900 50  0000 C CNN
+F 0 "R4" V 5943 3900 50  0000 C CNN
 F 1 "10k" V 6034 3900 50  0000 C CNN
 F 2 "" V 6080 3900 50  0001 C CNN
@@
 	6400 3900 6300 3900
 $Comp
-L keyboardParts:USB_mini_micro_B J?
+L keyboardParts:USB_mini_micro_B J1
 U 1 1 5F2509D5
 P 2000 3050
-F 0 "J?" H 1887 3341 60  0000 C CNN
+F 0 "J1" H 1887 3341 60  0000 C CNN
 F 1 "USB_mini_micro_B" H 1850 3300 60  0001 C CNN
 F 2 "" H 1950 3050 60  0000 C CNN
@@
 	2150 2900 2200 2900
 $Comp
-L power:VCC #PWR?
+L power:VCC #PWR0103
 U 1 1 5F25A61D
 P 2200 2850
-F 0 "#PWR?" H 2200 2700 50  0001 C CNN
+F 0 "#PWR0103" H 2200 2700 50  0001 C CNN
 F 1 "VCC" H 2215 3023 50  0000 C CNN
 F 2 "" H 2200 2850 50  0001 C CNN
@@
 	2200 2900 3450 2900
 $Comp
-L Device:R R?
+L Device:R R2
 U 1 1 5F25D0B4
 P 3200 3000
-F 0 "R?" V 2993 3000 50  0000 C CNN
+F 0 "R2" V 2993 3000 50  0000 C CNN
 F 1 "22" V 3084 3000 50  0000 C CNN
 F 2 "" V 3130 3000 50  0001 C CNN
@@
 $EndComp
 $Comp
-L Device:R R?
+L Device:R R3
 U 1 1 5F25F160
 P 3200 3100
-F 0 "R?" V 2993 3100 50  0000 C CNN
+F 0 "R3" V 2993 3100 50  0000 C CNN
 F 1 "22" V 3084 3100 50  0000 C CNN
 F 2 "" V 3130 3100 50  0001 C CNN
@@
 	2150 3100 3050 3100
 $Comp
-L Device:C C?
+L Device:C C8
 U 1 1 5F2675E8
 P 3200 3300
-F 0 "C?" V 2948 3300 50  0000 C CNN
+F 0 "C8" V 2948 3300 50  0000 C CNN
 F 1 "1u" V 3039 3300 50  0000 C CNN
 F 2 "" H 3238 3150 50  0001 C CNN
@@
 Connection ~ 2200 3300
 $Comp
-L power:GND #PWR?
+L power:GND #PWR0104
 U 1 1 5F2889A9
 P 1400 1950
-F 0 "#PWR?" H 1400 1700 50  0001 C CNN
+F 0 "#PWR0104" H 1400 1700 50  0001 C CNN
 F 1 "GND" H 1405 1777 50  0000 C CNN
 F 2 "" H 1400 1950 50  0001 C CNN
@@
 Connection ~ 1400 1900
 $Comp
-L power:GND #PWR?
+L power:GND #PWR0105
 U 1 1 5F28C864
 P 2950 3200
-F 0 "#PWR?" H 2950 2950 50  0001 C CNN
+F 0 "#PWR0105" H 2950 2950 50  0001 C CNN
 F 1 "GND" V 2955 3072 50  0000 R CNN
 F 2 "" H 2950 3200 50  0001 C CNN
@@
 $EndComp
 $Comp
-L power:GND #PWR?
+L power:GND #PWR0106
 U 1 1 5F28F081
 P 2400 4950
-F 0 "#PWR?" H 2400 4700 50  0001 C CNN
+F 0 "#PWR0106" H 2400 4700 50  0001 C CNN
 F 1 "GND" H 2405 4777 50  0000 C CNN
 F 2 "" H 2400 4950 50  0001 C CNN
@@
 $EndComp
 $Comp
-L power:GND #PWR?
+L power:GND #PWR0107
 U 1 1 5F291F0D
 P 6400 3900
-F 0 "#PWR?" H 6400 3650 50  0001 C CNN
+F 0 "#PWR0107" H 6400 3650 50  0001 C CNN
 F 1 "GND" V 6405 3772 50  0000 R CNN
 F 2 "" H 6400 3900 50  0001 C CNN
@@
 $EndComp
 $Comp
-L power:VCC #PWR?
+L power:VCC #PWR0108
 U 1 1 5F299AFB
 P 5600 2800
-F 0 "#PWR?" H 5600 2650 50  0001 C CNN
+F 0 "#PWR0108" H 5600 2650 50  0001 C CNN
 F 1 "VCC" V 5615 2928 50  0000 L CNN
 F 2 "" H 5600 2800 50  0001 C CNN
@@
 $EndComp
 $Comp
-L power:GND #PWR?
+L power:GND #PWR0109
 U 1 1 5F29C52D
 P 5600 2900
-F 0 "#PWR?" H 5600 2650 50  0001 C CNN
+F 0 "#PWR0109" H 5600 2650 50  0001 C CNN
 F 1 "GND" V 5605 2772 50  0000 R CNN
 F 2 "" H 5600 2900 50  0001 C CNN
@@
 $EndComp
 $Comp
-L power:GND #PWR?
+L power:GND #PWR0110
 U 1 1 5F29D224
 P 5600 3700
-F 0 "#PWR?" H 5600 3450 50  0001 C CNN
+F 0 "#PWR0110" H 5600 3450 50  0001 C CNN
 F 1 "GND" V 5605 3572 50  0000 R CNN
 F 2 "" H 5600 3700 50  0001 C CNN
@@
 $EndComp
 $Comp
-L power:VCC #PWR?
+L power:VCC #PWR0111
 U 1 1 5F2A2F72
 P 5600 3800
-F 0 "#PWR?" H 5600 3650 50  0001 C CNN
+F 0 "#PWR0111" H 5600 3650 50  0001 C CNN
 F 1 "VCC" V 5615 3928 50  0000 L CNN
 F 2 "" H 5600 3800 50  0001 C CNN
@@
 	5600 3900 6000 3900
 $Comp
-L power:GND #PWR?
+L power:GND #PWR0112
 U 1 1 5F2A4F0F
 P 5600 4900
-F 0 "#PWR?" H 5600 4650 50  0001 C CNN
+F 0 "#PWR0112" H 5600 4650 50  0001 C CNN
 F 1 "GND" V 5605 4772 50  0000 R CNN
 F 2 "" H 5600 4900 50  0001 C CNN
@@
 $EndComp
 $Comp
-L power:VCC #PWR?
+L power:VCC #PWR0113
 U 1 1 5F2A53B3
 P 5600 4800
-F 0 "#PWR?" H 5600 4650 50  0001 C CNN
+F 0 "#PWR0113" H 5600 4650 50  0001 C CNN
 F 1 "VCC" V 5615 4928 50  0000 L CNN
 F 2 "" H 5600 4800 50  0001 C CNN
@@
 $EndComp
 $Comp
-L power:GND #PWR?
+L power:GND #PWR0114
 U 1 1 5F2A6AED
 P 3450 4200
-F 0 "#PWR?" H 3450 3950 50  0001 C CNN
+F 0 "#PWR0114" H 3450 3950 50  0001 C CNN
 F 1 "GND" V 3455 4072 50  0000 R CNN
 F 2 "" H 3450 4200 50  0001 C CNN
@@
 $EndComp
 $Comp
-L power:VCC #PWR?
+L power:VCC #PWR0115
 U 1 1 5F2A73EA
 P 3450 4100
-F 0 "#PWR?" H 3450 3950 50  0001 C CNN
+F 0 "#PWR0115" H 3450 3950 50  0001 C CNN
 F 1 "VCC" V 3465 4227 50  0000 L CNN
 F 2 "" H 3450 4100 50  0001 C CNN
@@
 $EndComp
 $Comp
-L power:VCC #PWR?
+L power:VCC #PWR0116
 U 1 1 5F2A8035
 P 3450 3400
-F 0 "#PWR?" H 3450 3250 50  0001 C CNN
+F 0 "#PWR0116" H 3450 3250 50  0001 C CNN
 F 1 "VCC" V 3465 3527 50  0000 L CNN
 F 2 "" H 3450 3400 50  0001 C CNN
@@
 NoConn ~ 5600 3600
 $Comp
-L power:GND #PWR?
+L power:GND #PWR0117
 U 1 1 5F2FC66A
 P 2000 4000
-F 0 "#PWR?" H 2000 3750 50  0001 C CNN
+F 0 "#PWR0117" H 2000 3750 50  0001 C CNN
 F 1 "GND" V 2005 3872 50  0000 R CNN
 F 2 "" H 2000 4000 50  0001 C CNN
